File: documentation/eagle/timer2.sch (EAGLE design)
At the start: 8 parts

Commit message: version 1.1-2
Parts:
- removed U$1: NANO, Arduino-clone:NANO
- added U1: ATTINY85SU, attiny85:ATTINY85SU
- BATT: value 9V -> 4.5-5.5V
Connections:
- removed net N$2: R1.A, TM1637-3.S, U$1.5.5V
- net N$10: now also U1.PB3; no longer U$1.D4
- net N$12: now also R1.A, TM1637-3.S, U1.VCC; no longer U$1.RAW
- net N$3: now also U1.GND; no longer U$1.GND
- net N$5: no longer U$1.GND2
- net N$6: now also U1.PB0; no longer U$1.D2
- net N$7: now also U1.PB1; no longer U$1.D9
- net N$8: now also U1.PB2; no longer U$1.A0
- net N$9: now also U1.PB4; no longer U$1.D5
Changed lines of the file:
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@@
 <parts>
 <part name="SG1" library="buzzer" library_urn="urn:adsk.eagle:library:113" deviceset="B/C14L" device="" package3d_urn="urn:adsk.eagle:package:5281/1"/>
-<part name="BATT" library="SparkFun-Connectors" library_urn="urn:adsk.eagle:library:513" deviceset="BC9VPC" device="" package3d_urn="urn:adsk.eagle:package:38011/1" value=" 9V"/>
+<part name="BATT" library="SparkFun-Connectors" library_urn="urn:adsk.eagle:library:513" deviceset="BC9VPC" device="" package3d_urn="urn:adsk.eagle:package:38011/1" value="4.5-5.5V"/>
 <part name="TM1637" library="con-molex" library_urn="urn:adsk.eagle:library:165" deviceset="22-?-04" device="27-2041"/>
 <part name="R1" library="pot" library_urn="urn:adsk.eagle:library:331" deviceset="3RP/1610N" device="" package3d_urn="urn:adsk.eagle:package:22726/1" value="10k"/>
 <part name="S2PUSH-BUTTON" library="SparkFun-Switches" library_urn="urn:adsk.eagle:library:535" deviceset="MOMENTARY-SWITCH-SPST" device="-PTH-6.0MM" package3d_urn="urn:adsk.eagle:package:40163/1" value=""/>
 <part name="S1ON-OFF" library="SparkFun-Switches" library_urn="urn:adsk.eagle:library:535" deviceset="MOMENTARY-SWITCH-SPST" device="-PTH-6.0MM" package3d_urn="urn:adsk.eagle:package:40163/1" value=""/>
-<part name="U$1" library="Arduino-clone" deviceset="NANO" device=""/>
 <part name="R2" library="eagle-ltspice" library_urn="urn:adsk.eagle:library:217" deviceset="R" device="0204/7" package3d_urn="urn:adsk.eagle:package:13274/1" value="220"/>
+<part name="U1" library="attiny85" deviceset="ATTINY85" device="SU"/>
 </parts>
 <sheets>
@@
 <instance part="S2PUSH-BUTTON" gate="G$1" x="71.12" y="86.36"/>
 <instance part="S1ON-OFF" gate="G$1" x="-17.78" y="91.44"/>
-<instance part="U$1" gate="G$1" x="33.02" y="68.58"/>
 <instance part="R2" gate="G$1" x="53.34" y="76.2"/>
+<instance part="U1" gate="G$1" x="25.4" y="43.18"/>
 </instances>
 <busses>
@@
 </segment>
 </net>
-<net name="N$2" class="0">
-<segment>
-<pinref part="U$1" gate="G$1" pin="5.5V"/>
-<pinref part="R1" gate="G$1" pin="A"/>
-<wire x1="-10.16" y1="55.88" x2="-2.54" y2="55.88" width="0.1524" layer="91"/>
-<wire x1="-2.54" y1="55.88" x2="10.16" y2="55.88" width="0.1524" layer="91"/>
-<wire x1="-2.54" y1="63.5" x2="-2.54" y2="55.88" width="0.1524" layer="91"/>
-<junction x="-2.54" y="55.88"/>
-<pinref part="TM1637" gate="-3" pin="S"/>
-<wire x1="50.8" y1="20.32" x2="-10.16" y2="20.32" width="0.1524" layer="91"/>
-<wire x1="-10.16" y1="20.32" x2="-10.16" y2="55.88" width="0.1524" layer="91"/>
-</segment>
-</net>
 <net name="N$3" class="0">
 <segment>
@@
 <wire x1="-7.62" y1="48.26" x2="0" y2="48.26" width="0.1524" layer="91"/>
 <wire x1="0" y1="48.26" x2="0" y2="50.8" width="0.1524" layer="91"/>
-<pinref part="U$1" gate="G$1" pin="GND"/>
 <wire x1="0" y1="50.8" x2="10.16" y2="50.8" width="0.1524" layer="91"/>
 <pinref part="R1" gate="G$1" pin="E"/>
@@
 <wire x1="-15.24" y1="15.24" x2="-15.24" y2="48.26" width="0.1524" layer="91"/>
 <junction x="-15.24" y="48.26"/>
+<pinref part="U1" gate="G$1" pin="GND"/>
+<wire x1="10.16" y1="50.8" x2="10.16" y2="35.56" width="0.1524" layer="91"/>
 </segment>
 </net>
@@
 <segment>
 <pinref part="SG1" gate="G$1" pin="2"/>
-<pinref part="U$1" gate="G$1" pin="GND2"/>
 <wire x1="68.58" y1="63.5" x2="68.58" y2="55.88" width="0.1524" layer="91"/>
 <wire x1="68.58" y1="55.88" x2="60.96" y2="55.88" width="0.1524" layer="91"/>
 <pinref part="S2PUSH-BUTTON" gate="G$1" pin="2"/>
-<wire x1="60.96" y1="55.88" x2="43.18" y2="55.88" width="0.1524" layer="91"/>
 <wire x1="76.2" y1="86.36" x2="81.28" y2="86.36" width="0.1524" layer="91"/>
 <wire x1="81.28" y1="86.36" x2="81.28" y2="91.44" width="0.1524" layer="91"/>
 <wire x1="81.28" y1="91.44" x2="60.96" y2="91.44" width="0.1524" layer="91"/>
 <wire x1="60.96" y1="91.44" x2="60.96" y2="55.88" width="0.1524" layer="91"/>
-<junction x="60.96" y="55.88"/>
 </segment>
 </net>
 <net name="N$6" class="0">
 <segment>
-<pinref part="U$1" gate="G$1" pin="D2"/>
-<wire x1="43.18" y1="58.42" x2="66.04" y2="58.42" width="0.1524" layer="91"/>
 <pinref part="S2PUSH-BUTTON" gate="G$1" pin="1"/>
-<wire x1="66.04" y1="58.42" x2="66.04" y2="86.36" width="0.1524" layer="91"/>
+<wire x1="66.04" y1="35.56" x2="66.04" y2="86.36" width="0.1524" layer="91"/>
+<pinref part="U1" gate="G$1" pin="PB0"/>
+<wire x1="43.18" y1="35.56" x2="66.04" y2="35.56" width="0.1524" layer="91"/>
 </segment>
 </net>
 <net name="N$8" class="0">
 <segment>
-<pinref part="U$1" gate="G$1" pin="A0"/>
 <pinref part="R1" gate="G$1" pin="S"/>
-<wire x1="10.16" y1="76.2" x2="2.54" y2="76.2" width="0.1524" layer="91"/>
 <wire x1="2.54" y1="76.2" x2="2.54" y2="68.58" width="0.1524" layer="91"/>
-</segment>
-</net>
-<net name="N$9" class="0">
-<segment>
-<pinref part="TM1637" gate="-1" pin="S"/>
-<wire x1="50.8" y1="30.48" x2="50.8" y2="66.04" width="0.1524" layer="91"/>
-<pinref part="U$1" gate="G$1" pin="D5"/>
-<wire x1="50.8" y1="66.04" x2="43.18" y2="66.04" width="0.1524" layer="91"/>
+<wire x1="2.54" y1="76.2" x2="27.94" y2="76.2" width="0.1524" layer="91"/>
+<wire x1="27.94" y1="76.2" x2="27.94" y2="63.5" width="0.1524" layer="91"/>
+<wire x1="27.94" y1="63.5" x2="53.34" y2="63.5" width="0.1524" layer="91"/>
+<wire x1="53.34" y1="63.5" x2="53.34" y2="40.64" width="0.1524" layer="91"/>
+<pinref part="U1" gate="G$1" pin="PB2"/>
+<wire x1="53.34" y1="40.64" x2="43.18" y2="40.64" width="0.1524" layer="91"/>
 </segment>
 </net>
@@
 <segment>
 <pinref part="TM1637" gate="-2" pin="S"/>
-<wire x1="50.8" y1="25.4" x2="45.72" y2="25.4" width="0.1524" layer="91"/>
-<wire x1="45.72" y1="25.4" x2="45.72" y2="63.5" width="0.1524" layer="91"/>
-<pinref part="U$1" gate="G$1" pin="D4"/>
-<wire x1="45.72" y1="63.5" x2="43.18" y2="63.5" width="0.1524" layer="91"/>
+<pinref part="U1" gate="G$1" pin="PB3"/>
+<wire x1="43.18" y1="43.18" x2="50.8" y2="43.18" width="0.1524" layer="91"/>
+<wire x1="50.8" y1="43.18" x2="50.8" y2="25.4" width="0.1524" layer="91"/>
 </segment>
 </net>
@@
 <segment>
 <pinref part="R2" gate="G$1" pin="1"/>
-<pinref part="U$1" gate="G$1" pin="D9"/>
 <wire x1="48.26" y1="76.2" x2="43.18" y2="76.2" width="0.1524" layer="91"/>
+<wire x1="43.18" y1="76.2" x2="43.18" y2="53.34" width="0.1524" layer="91"/>
+<wire x1="43.18" y1="53.34" x2="48.26" y2="53.34" width="0.1524" layer="91"/>
+<wire x1="48.26" y1="53.34" x2="48.26" y2="38.1" width="0.1524" layer="91"/>
+<pinref part="U1" gate="G$1" pin="PB1"/>
+<wire x1="48.26" y1="38.1" x2="43.18" y2="38.1" width="0.1524" layer="91"/>
 </segment>
 </net>
@@
 <pinref part="S1ON-OFF" gate="G$1" pin="2"/>
 <wire x1="-12.7" y1="91.44" x2="5.08" y2="91.44" width="0.1524" layer="91"/>
-<pinref part="U$1" gate="G$1" pin="RAW"/>
 <wire x1="5.08" y1="91.44" x2="5.08" y2="48.26" width="0.1524" layer="91"/>
 <wire x1="5.08" y1="48.26" x2="10.16" y2="48.26" width="0.1524" layer="91"/>
+<pinref part="U1" gate="G$1" pin="VCC"/>
+<pinref part="R1" gate="G$1" pin="A"/>
+<wire x1="-10.16" y1="55.88" x2="-2.54" y2="55.88" width="0.1524" layer="91"/>
+<wire x1="-2.54" y1="63.5" x2="-2.54" y2="55.88" width="0.1524" layer="91"/>
+<pinref part="TM1637" gate="-3" pin="S"/>
+<wire x1="50.8" y1="20.32" x2="5.08" y2="20.32" width="0.1524" layer="91"/>
+<wire x1="5.08" y1="20.32" x2="-10.16" y2="20.32" width="0.1524" layer="91"/>
+<wire x1="-10.16" y1="20.32" x2="-10.16" y2="55.88" width="0.1524" layer="91"/>
+<wire x1="5.08" y1="48.26" x2="5.08" y2="20.32" width="0.1524" layer="91"/>
+<junction x="5.08" y="48.26"/>
+<junction x="5.08" y="20.32"/>
 </segment>
 </net>
+<net name="N$9" class="0">
+<segment>
+<pinref part="TM1637" gate="-1" pin="S"/>
+<wire x1="50.8" y1="30.48" x2="45.72" y2="30.48" width="0.1524" layer="91"/>
+<wire x1="45.72" y1="30.48" x2="45.72" y2="45.72" width="0.1524" layer="91"/>
+<pinref part="U1" gate="G$1" pin="PB4"/>
+<wire x1="45.72" y1="45.72" x2="43.18" y2="45.72" width="0.1524" layer="91"/>
+</segment>
+</net>
