File: documentation/eagle/timer2.sch (EAGLE design)
At the start: 8 parts, among them U1 ATTINY85SU

Commit message: updating documentation
Parts:
- added C1: 100nF, resistor:C-EU025-024X044
Connections:
- net N$3: now also C1.2
Changed lines of the file:
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@@
 <part name="R2" library="eagle-ltspice" library_urn="urn:adsk.eagle:library:217" deviceset="R" device="0204/7" package3d_urn="urn:adsk.eagle:package:13274/1" value="220"/>
 <part name="U1" library="attiny85" deviceset="ATTINY85" device="SU"/>
+<part name="C1" library="resistor" library_urn="urn:adsk.eagle:library:348" deviceset="C-EU" device="025-024X044" package3d_urn="urn:adsk.eagle:package:26149/1" value="100nF"/>
 </parts>
 <sheets>
@@
 <instance part="R2" gate="G$1" x="53.34" y="76.2"/>
 <instance part="U1" gate="G$1" x="25.4" y="43.18"/>
+<instance part="C1" gate="G$1" x="12.7" y="45.72"/>
 </instances>
 <busses>
@@
 <junction x="-15.24" y="48.26"/>
 <pinref part="U1" gate="G$1" pin="GND"/>
-<wire x1="10.16" y1="50.8" x2="10.16" y2="35.56" width="0.1524" layer="91"/>
+<wire x1="10.16" y1="50.8" x2="10.16" y2="40.64" width="0.1524" layer="91"/>
+<wire x1="10.16" y1="40.64" x2="10.16" y2="35.56" width="0.1524" layer="91"/>
 <wire x1="2.54" y1="50.8" x2="2.54" y2="58.42" width="0.1524" layer="91"/>
 <junction x="2.54" y="50.8"/>
@@
 <wire x1="2.54" y1="58.42" x2="60.96" y2="58.42" width="0.1524" layer="91"/>
 <junction x="60.96" y="58.42"/>
+<pinref part="C1" gate="G$1" pin="2"/>
+<wire x1="12.7" y1="40.64" x2="10.16" y2="40.64" width="0.1524" layer="91"/>
+<junction x="10.16" y="40.64"/>
 </segment>
 </net>
